File: leds.kicad_sch (KiCad schematic)
At the start: 0 parts

Commit message: Place the 12 LEDs in one straight line at 10 mm pitch.
Parts:
- added D1, D10, D11, D12, D2, D3, D4, D5, D6, D7, D8, D9: LED_CV28, CV28D-FCC:LED_CV28, symbol LED_CV28:LED_CV28
Connections:
- new net: D8.1 (B_C), D9.6 (B_A)
- new net: D8.2 (G_C), D9.5 (G_A)
- new net: D8.3 (R_C), D9.4 (R_A)
- new net: D7.3 (R_C), D8.4 (R_A)
- new net: D7.2 (G_C), D8.5 (G_A)
- new net: D7.1 (B_C), D8.6 (B_A)
- new net: D2.3 (R_C), D3.4 (R_A)
- new net: D2.2 (G_C), D3.5 (G_A)
- new net: D2.1 (B_C), D3.6 (B_A)
- new net: D5.1 (B_C), D6.6 (B_A)
- new net: D5.2 (G_C), D6.5 (G_A)
- new net: D5.3 (R_C), D6.4 (R_A)
- new net: D4.3 (R_C), D5.4 (R_A)
- new net: D4.2 (G_C), D5.5 (G_A)
- new net: D4.1 (B_C), D5.6 (B_A)
- new net: D10.1 (B_C), D11.6 (B_A)
- new net: D10.2 (G_C), D11.5 (G_A)
- new net: D10.3 (R_C), D11.4 (R_A)
- new net: D11.3 (R_C), D12.4 (R_A)
- new net: D11.2 (G_C), D12.5 (G_A)
- new net: D11.1 (B_C), D12.6 (B_A)
- new net: D1.1 (B_C), D2.6 (B_A)
- new net: D1.2 (G_C), D2.5 (G_A)
- new net: D1.3 (R_C), D2.4 (R_A)
- new net +12V: D1.4 (R_A), D1.5 (G_A), D1.6 (B_A), D10.4 (R_A), D10.5 (G_A), D10.6 (B_A), D4.4 (R_A), D4.5 (G_A), D4.6 (B_A), D7.4 (R_A), D7.5 (G_A), D7.6 (B_A)
- new net OUT0_R0: D3.3 (R_C)
- new net OUT10_B2: D9.1 (B_C)
- new net OUT11_B3: D12.1 (B_C)
- new net OUT1_R1: D6.3 (R_C)
- new net OUT2_R2: D9.3 (R_C)
- new net OUT3_R3: D12.3 (R_C)
- new net OUT4_G0: D3.2 (G_C)
- new net OUT5_G1: D6.2 (G_C)
- new net OUT6_G2: D9.2 (G_C)
- new net OUT7_G3: D12.2 (G_C)
- new net OUT8_B0: D3.1 (B_C)
- new net OUT9_B1: D6.1 (B_C)
